File: Driver.kicad_pcb (KiCad board)
At the start: 2 copper layers, 25.5 x 40.5 mm, 16 parts, among them J1 Conn_01x05_Socket, J2 Conn_01x05_Socket, J3 Conn_01x05_Pin, U1 IS31FL3239

Commit message: Final RevA Board
Parts:
- added kibuzzard-64D44BAC: G***, kibuzzard-64D44BAC, B.Cu at (195.2, 82.0)
- added kibuzzard-64D44BB9: G***, kibuzzard-64D44BB9, B.Cu at (197.7, 82.0)
- added kibuzzard-64D44BBD: G***, kibuzzard-64D44BBD, B.Cu at (200.2, 82.0)
- added kibuzzard-64D44BC4: G***, kibuzzard-64D44BC4, B.Cu at (202.8, 82.0)
- added kibuzzard-64D44BC8: G***, kibuzzard-64D44BC8, B.Cu at (205.3, 82.0)

Commit message: Updated I2C addresses to correct one on silkscreen
Other:
- board text added: "0x34"
- board text added: "0x35"
- board text added: "0x36"
- board text added: "0x37"
- board text removed: "0x44"
- board text removed: "0x45"
- board text removed: "0x46"
- board text removed: "0x47"
Changed lines of the file:
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@@
   (gr_line (start 213 118) (end 187.5 118)
     (stroke (width 0.1) (type default)) (layer "Edge.Cuts"))
-  (gr_text "0x44" (at 201 92.25 90) (layer "B.SilkS")
+  (gr_text "0x34" (at 201 92.25 90) (layer "B.SilkS")
     (effects (font (size 0.6 0.6) (thickness 0.09)) (justify mirror))
   )
@@
     (effects (font (size 1 1) (thickness 0.125)) (justify bottom mirror))
   )
-  (gr_text "0x45" (at 202 92.25 90) (layer "B.SilkS")
+  (gr_text "0x35" (at 202 92.25 90) (layer "B.SilkS")
     (effects (font (size 0.6 0.6) (thickness 0.09)) (justify mirror))
   )
-  (gr_text "0x46" (at 202 89.75 90) (layer "B.SilkS")
+  (gr_text "0x36" (at 202 89.75 90) (layer "B.SilkS")
     (effects (font (size 0.6 0.6) (thickness 0.09)) (justify mirror))
   )
@@
     (effects (font (size 0.75 0.75) (thickness 0.1)) (justify right bottom mirror))
   )
-  (gr_text "0x47" (at 201 89.75 90) (layer "B.SilkS")
+  (gr_text "0x37" (at 201 89.75 90) (layer "B.SilkS")
     (effects (font (size 0.6 0.6) (thickness 0.09)) (justify mirror))
   )
@@
     (pts (xy 213 77.5) (xy 213 118))
     (height -4.5)
-    (gr_text "40.5000 mm" (at 216.35 97.75 90) (layer "User.2")
+    (gr_text "1594.4882 mils" (at 216.35 97.75 90) (layer "User.2")
       (effects (font (size 1 1) (thickness 0.15)))
     )
@@
     (pts (xy 187.5 77.5) (xy 213 77.5))
     (height -10)
-    (gr_text "25.5000 mm" (at 200.25 66.35) (layer "User.2")
+    (gr_text "1003.9370 mils" (at 200.25 66.35) (layer "User.2")
       (effects (font (size 1 1) (thickness 0.15)))
     )
@@
     (pts (xy 213 77.5) (xy 213 97.75))
     (height -1.5)
-    (gr_text "20.2500 mm" (at 213.35 87.625 90) (layer "User.2")
+    (gr_text "797.2441 mils" (at 213.35 87.625 90) (layer "User.2")
       (effects (font (size 1 1) (thickness 0.15)))
     )
@@
     (pts (xy 213 77.5) (xy 200.25 77.5))
     (height 7.5)
-    (gr_text "12.7500 mm" (at 206.625 68.85) (layer "User.2")
+    (gr_text "501.9685 mils" (at 206.625 68.85) (layer "User.2")
       (effects (font (size 1 1) (thickness 0.15)))
     )
